Commit message: Attempt 4 lol.

File: assembly/urdf/quad/urdf/quad.urdf (robot description, URDF)
Before this commit: robot quad, 13 links, 12 joints
Links:
- link bl_calf: mass 0.41885 -> 0.41885250755801
- link bl_foot: mass 0.12868 -> 0.128682263244567
- link bl_thigh: mass 0.37562 -> 0.375618459455155
- link body: mass 0.54938 -> 2.2513
- link br_calf: mass 0.41885 -> 0.418852507558011
- link br_foot: mass 0.12868 -> 0.128682263244567
- link br_thigh: mass 0.37562 -> 0.375618459455154
- link fl_calf: mass 0.41885 -> 0.41885250755801
- link fl_foot: mass 0.12868 -> 0.128682263244567
- link fr_calf: mass 0.41885 -> 0.418852507558011
- link fr_foot: mass 0.12868 -> 0.128682263244566
- link fr_thigh: mass 0.37562 -> 0.375618459455155
Joints:
- joint bl_hip_pitch: axis 0 1 0 -> 0 -1 0; limit lower=-12.56 upper=12.56 effort=10 velocity=0 -> lower=-12.56 upper=12.56 effort=10 velocity=250
- joint bl_hip_roll: axis 1 0 0 -> -1 0 0; limit lower=-12.56 upper=12.56 effort=10 velocity=0 -> lower=-12.56 upper=12.56 effort=10 velocity=250
- joint bl_knee_pitch: axis 0 1 0 -> 0 -1 0; limit lower=-12.56 upper=12.56 effort=10 velocity=0 -> lower=-12.56 upper=12.56 effort=10 velocity=250
- joint br_hip_pitch: axis 0 -1 0 -> 0 1 0; limit lower=-12.56 upper=12.56 effort=10 velocity=0 -> lower=-12.56 upper=12.56 effort=10 velocity=250
- joint br_hip_roll: axis -1 0 0 -> 1 0 0; limit lower=-12.56 upper=12.56 effort=10 velocity=0 -> lower=-12.56 upper=12.56 effort=10 velocity=250
- joint br_knee_pitch: axis 0 -1 0 -> 0 1 0; limit lower=-12.56 upper=12.56 effort=10 velocity=0 -> lower=-12.56 upper=12.56 effort=10 velocity=250
- joint fl_hip_pitch: axis 0 1 0 -> 0 -1 0; limit lower=-12.56 upper=12.56 effort=10 velocity=0 -> lower=-12.56 upper=12.56 effort=10 velocity=250
- joint fl_hip_roll: axis 1 0 0 -> -1 0 0; limit lower=-12.56 upper=12.56 effort=10 velocity=0 -> lower=-12.56 upper=12.56 effort=10 velocity=250
- joint fl_knee_pitch: axis 0 1 0 -> 0 -1 0; limit lower=-12.56 upper=12.56 effort=10 velocity=0 -> lower=-12.56 upper=12.56 effort=10 velocity=250
- joint fr_hip_pitch: axis 0 -1 0 -> 0 1 0; limit lower=-12.56 upper=12.56 effort=10 velocity=0 -> lower=-12.56 upper=12.56 effort=10 velocity=250
- joint fr_hip_roll: axis -1 0 0 -> 1 0 0; limit lower=-12.56 upper=12.56 effort=10 velocity=0 -> lower=-12.56 upper=12.56 effort=10 velocity=250
- joint fr_knee_pitch: axis 0 -1 0 -> 0 1 0; limit lower=-12.56 upper=12.56 effort=10 velocity=0 -> lower=-12.56 upper=12.56 effort=10 velocity=250

Commit message: Regenerated quad with inward legs.

File: assembly/urdf/quad/urdf/quad.urdf (robot description, URDF)
Before this commit: robot quad, 13 links, 12 joints
Links:
- link body: mass 2.2513 -> 2.25128521088266
- link br_foot: mass 0.128682263244567 -> 0.12868
- link br_thigh: mass 0.375618459455154 -> 0
- link fr_calf: mass 0.418852507558011 -> 0.41885250755801
Joints:
- joint bl_hip_pitch: axis 0 -1 0 -> 0 1 0
- joint bl_hip_roll: axis -1 0 0 -> 1 0 0
- joint bl_knee_pitch: axis 0 -1 0 -> 0 1 0
- joint br_hip_pitch: axis 0 1 0 -> 0 -1 0
- joint br_hip_roll: axis 1 0 0 -> -1 0 0
- joint br_knee_pitch: axis 0 1 0 -> 0 -1 0
- joint fl_hip_pitch: axis 0 -1 0 -> 0 1 0
- joint fl_hip_roll: axis -1 0 0 -> 1 0 0
- joint fl_knee_pitch: axis 0 -1 0 -> 0 1 0
- joint fr_hip_pitch: axis 0 1 0 -> 0 -1 0
- joint fr_hip_roll: axis 1 0 0 -> -1 0 0
- joint fr_knee_pitch: axis 0 1 0 -> 0 -1 0

Commit message: Short urdf.

File: assembly/urdf/quad/urdf/quad.urdf (robot description, URDF)
Before this commit: robot quad, 13 links, 12 joints
Links:
- link bl_calf: mass 0.41885250755801 -> 0.369733221029887
- link bl_foot: mass 0.128682263244567 -> 0.113203575524731
- link bl_thigh: mass 0.375618459455155 -> 0.32829098650712
- link body: mass 2.25128521088266 -> 0.688615038914901
- link br_calf: mass 0.418852507558011 -> 0.369733221029887
- link br_foot: mass 0.128682263244567 -> 0.113203575524731
- link br_thigh: mass 0.375618459455154 -> 0.32829098650712
- link fl_calf: mass 0.41885250755801 -> 0.369733221029888
- link fl_foot: mass 0.128682263244567 -> 0.113203575524731
- link fl_thigh: mass 0.375618459455155 -> 0.32829098650712
- link fr_calf: mass 0.418852507558011 -> 0.369733221029888
- link fr_foot: mass 0.128682263244566 -> 0.113203575524731
- link fr_thigh: mass 0.375618459455155 -> 0.32829098650712
Joints:
- joint bl_hip_pitch: origin xyz=-0.19225 0.023 0 rpy=0 0 0 -> xyz=-0.25125 -0.016 0 rpy=0 0 0
- joint bl_hip_roll: origin xyz=-0.441 0.11772 0 rpy=0 0 0 -> xyz=-0.295 0.11772 -0.00011829 rpy=0 0 0
- joint bl_knee_pitch: origin xyz=0 0.081 -0.19625 rpy=0 0 0 -> xyz=0 0.063 -0.15625 rpy=0 0 0
- joint br_hip_pitch: origin xyz=-0.19225 -0.023 0 rpy=0 0 0 -> xyz=-0.19925 0.016 0 rpy=0 0 0
- joint br_hip_roll: origin xyz=-0.441 -0.11773 0 rpy=0 0 0 -> xyz=-0.347 -0.11773 -0.00011829 rpy=0 0 0
- joint br_knee_pitch: origin xyz=0 -0.081 -0.19625 rpy=0 0 0 -> xyz=0 -0.063 -0.15625 rpy=0 0 0
- joint fl_hip_pitch: origin xyz=0.19225 0.023 0 rpy=0 0 0 -> xyz=0.19925 -0.016 0 rpy=0 0 0
- joint fl_hip_roll: origin xyz=-0.214 0.11772 0 rpy=0 0 0 -> xyz=-0.221 0.11772 -0.00011829 rpy=0 0 0
- joint fl_knee_pitch: origin xyz=0 0.081 -0.19625 rpy=0 0 0 -> xyz=0 0.063 -0.15625 rpy=0 0 0
- joint fr_hip_pitch: origin xyz=0.19225 -0.023 0 rpy=0 0 0 -> xyz=0.25125 0.016 0 rpy=0 0 0
- joint fr_hip_roll: origin xyz=-0.214 -0.11773 0 rpy=0 0 0 -> xyz=-0.273 -0.11773 -0.00011829 rpy=0 0 0
- joint fr_knee_pitch: origin xyz=0 -0.081 -0.19625 rpy=0 0 0 -> xyz=0 -0.063 -0.15625 rpy=0 0 0

Commit message: Added hips to body in urdf.

File: assembly/urdf/quad/urdf/quad.urdf (robot description, URDF)
Before this commit: robot quad, 13 links, 12 joints
Links:
- link body: mass 0.688615038914901 -> 2.38478530150357
- link br_calf: mass 0.369733221029887 -> 0.369733221029888
Joints:
- joint bl_hip_pitch: origin xyz=-0.25125 -0.016 0 rpy=0 0 0 -> xyz=-0.26788 -0.016 0 rpy=0 0 0
- joint bl_hip_roll: origin xyz=-0.295 0.11772 -0.00011829 rpy=0 0 0 -> xyz=-0.011 0.055225 -0.04425 rpy=0 0 0
- joint br_hip_pitch: origin xyz=-0.19925 0.016 0 rpy=0 0 0 -> xyz=-0.21018 0.016 0 rpy=0 0 0
- joint br_hip_roll: origin xyz=-0.347 -0.11773 -0.00011829 rpy=0 0 0 -> xyz=-0.063 -0.18022 -0.04425 rpy=0 0 0
- joint fl_hip_pitch: origin xyz=0.19925 -0.016 0 rpy=0 0 0 -> xyz=0.22826 -0.016 0 rpy=0 0 0
- joint fl_hip_roll: origin xyz=-0.221 0.11772 -0.00011829 rpy=0 0 0 -> xyz=0.063 0.055225 -0.04425 rpy=0 0 0
- joint fr_hip_pitch: origin xyz=0.25125 0.016 0 rpy=0 0 0 -> xyz=0.2612 0.016 0 rpy=0 0 0
- joint fr_hip_roll: origin xyz=-0.273 -0.11773 -0.00011829 rpy=0 0 0 -> xyz=0.011 -0.18022 -0.04425 rpy=0 0 0

Commit message: Fixed coordinates.

File: assembly/urdf/quad/urdf/quad.urdf (robot description, URDF)
Before this commit: robot quad, 13 links, 12 joints
Joints:
- joint bl_hip_pitch: origin xyz=-0.26788 -0.016 0 rpy=0 0 0 -> xyz=-0.25125 -0.016 0 rpy=0 0 0
- joint br_hip_pitch: origin xyz=-0.21018 0.016 0 rpy=0 0 0 -> xyz=-0.19925 0.016 0 rpy=0 0 0
- joint fl_hip_pitch: origin xyz=0.22826 -0.016 0 rpy=0 0 0 -> xyz=0.19925 -0.016 0 rpy=0 0 0
- joint fr_hip_pitch: origin xyz=0.2612 0.016 0 rpy=0 0 0 -> xyz=0.25125 0.016 0 rpy=0 0 0
